Commit message: testing branch first commit

File: src/src/main_bot_description/urdf/main_bot_description.urdf.xacro (robot description, xacro)
@@ -9,10 +9,4 @@
   <xacro:property name="wheel_mass" value="0.5"/>
   <xacro:property name="base_mass" value="5.0"/>
-  <material name="grey">
-    <color rgba="0.5 0.5 0.5 1.0"/>
-  </material>
-  <material name="turquoise">
-    <color rgba="0.25 0.88 0.82 1.0"/>
-  </material>
   <!-- Base Link -->
   <link name="base_link">
@@ -32,5 +26,5 @@
     <inertial>
       <mass value="${base_mass}"/>
-      <inertia ixx="0.04167" ixy="0.0" ixz="0.0" iyy="0.10833" iyz="0.0" izz="0.14167"/>
+      <inertia ixx="1.0" ixy="0.0" ixz="0.0" iyy="1.0" iyz="0.0" izz="1.0"/>
     </inertial>
   </link>
@@ -66,5 +60,5 @@
         <cylinder radius="0.01" length="0.3"/>
       </geometry>
-      <material name="turquoise"/>
+      <material name="grey"/>
     </visual>
     <collision>
@@ -83,45 +77,16 @@
     <origin xyz="0 0 ${base_height}" rpy="0 0 0"/>
     <axis xyz="0 0 1"/>
-    <limit lower="0.0" upper="1" effort="10.0" velocity="0.1"/>
-    <dynamics damping="0.7"/>
+    <limit lower="0.0" upper="0.5" effort="10.0" velocity="0.1"/>
   </joint>
-  <ros2_control name="GazeboSystem" type="system">
-    <hardware>
-      <plugin>gazebo_ros2_control/GazeboSystem</plugin>
-    </hardware>
+  <transmission name="antenna_trans">
+    <type>transmission_interface/SimpleTransmission</type>
     <joint name="antenna_joint">
-      <command_interface name="position">
-        <param name="min">0.0</param>
-        <param name="max">0.5</param>
-      </command_interface>
-      <state_interface name="position"/>
-      <state_interface name="velocity"/>
+      <hardwareInterface>hardware_interface/PositionJointInterface</hardwareInterface>
     </joint>
-    <joint name="front_left_wheel_joint">
-        <command_interface name="velocity"/>
-        <state_interface name="position"/>
-        <state_interface name="velocity"/>
-    </joint>
-    <joint name="front_right_wheel_joint">
-        <command_interface name="velocity"/>
-        <state_interface name="position"/>
-        <state_interface name="velocity"/>
-    </joint>
-    <joint name="rear_left_wheel_joint">
-        <command_interface name="velocity"/>
-        <state_interface name="position"/>
-        <state_interface name="velocity"/>
-    </joint>
-    <joint name="rear_right_wheel_joint">
-        <command_interface name="velocity"/>
-        <state_interface name="position"/>
-        <state_interface name="velocity"/>
-    </joint>
-  </ros2_control>
-  <gazebo reference="base_link">
-    <mu1>0.8</mu1>
-    <mu2>0.8</mu2>
-    <material>Gazebo/Grey</material>
-  </gazebo>
+    <actuator name="antenna_motor">
+      <hardwareInterface>hardware_interface/PositionJointInterface</hardwareInterface>
+      <mechanicalReduction>1</mechanicalReduction>
+    </actuator>
+  </transmission>
   <!-- Wheel Macro -->
   <xacro:macro name="wheel" params="prefix x_offset y_offset">
@@ -145,9 +110,4 @@
       </inertial>
     </link>
-    <gazebo reference="${prefix}_wheel_link">
-        <mu1>1.0</mu1>
-        <mu2>1.0</mu2>
-        <material>Gazebo/Black</material>
-    </gazebo>
     <joint name="${prefix}_wheel_joint" type="continuous">
       <parent link="base_link"/>
@@ -184,5 +144,8 @@
       </ray>
       <plugin name="gazebo_ros_lidar_controller" filename="libgazebo_ros_ray_sensor.so">
-        <topic>/gazebo_ros_lidar_controller/out</topic>
+        <ros>
+            <namespace>/demo</namespace>
+            <argument>--ros-args --remap ~/out:=scan</argument>
+        </ros>
         <output_type>sensor_msgs/LaserScan</output_type>
         <frame_name>lidar_link</frame_name>
@@ -190,10 +153,20 @@
     </sensor>
   </gazebo>
-  <!-- Gazebo Plugin for ROS2 Control -->
+  <!-- Gazebo Plugin for Differential Drive -->
   <gazebo>
     <plugin name="gazebo_ros2_control" filename="libgazebo_ros2_control.so">
       <robot_param>robot_description</robot_param>
       <robot_param_node>robot_state_publisher</robot_param_node>
-      <parameters>/home/rakshaa/ros2_ws/src/src/main_bot_description/config/controllers.yaml</parameters>
+      <parameters>$(find main_bot_description)/config/controllers.yaml</parameters>
+    </plugin>
+    <plugin name="differential_drive_controller" filename="libgazebo_ros_diff_drive.so">
+      <left_joint>front_left_wheel_joint</left_joint>
+      <right_joint>front_right_wheel_joint</right_joint>
+      <wheel_separation>${base_width}</wheel_separation>
+      <wheel_diameter>${2*wheel_radius}</wheel_diameter>
+      <robot_base_frame>base_link</robot_base_frame>
+      <publish_odom>true</publish_odom>
+      <publish_odom_tf>true</publish_odom_tf>
+      <publish_wheel_tf>true</publish_wheel_tf>
     </plugin>
   </gazebo>
